File: LMFEmimicboard.sch (KiCad schematic (older format))
At the start: 9 parts, among them J1 D, J2 S, J3 F, J4 P, Q1 BF862

Commit message: Changed values to match the LMFE.
Parts:
- removed R2: 0, Resistor_SMD:R_0402_1005Metric, symbol Device:R
- C1: value C -> 0.35 pF
- C2: value C -> 0.1 pF
- R1: value 10k -> 1G
Changed lines of the file:
@@
 P 3850 2500
 F 0 "R1" V 3643 2500 50  0000 C CNN
-F 1 "10k" V 3734 2500 50  0000 C CNN
+F 1 "1G" V 3734 2500 50  0000 C CNN
 F 2 "Resistor_SMD:R_0402_1005Metric" V 3780 2500 50  0001 C CNN
 F 3 "~" H 3850 2500 50  0001 C CNN
@@
 Wire Wire Line
 	4600 1650 4600 2300
-$Comp
-L power:GND #PWR0103
-U 1 1 5F3F85EB
-P 5000 1700
-F 0 "#PWR0103" H 5000 1450 50  0001 C CNN
-F 1 "GND" H 5005 1527 50  0000 C CNN
-F 2 "" H 5000 1700 50  0001 C CNN
-F 3 "" H 5000 1700 50  0001 C CNN
-	1    5000 1700
-	1    0    0    -1
-$EndComp
-Wire Wire Line
-	4600 1650 4650 1650
-Connection ~ 4600 1650
-Wire Wire Line
-	4950 1650 5000 1650
-Wire Wire Line
-	5000 1650 5000 1700
 Connection ~ 4050 2850
 Wire Wire Line
@@
 $EndComp
 $Comp
-L Device:R R2
-U 1 1 5F3F7CD9
-P 4800 1650
-F 0 "R2" V 4593 1650 50  0000 C CNN
-F 1 "0" V 4684 1650 50  0000 C CNN
-F 2 "Resistor_SMD:R_0402_1005Metric" V 4730 1650 50  0001 C CNN
-F 3 "~" H 4800 1650 50  0001 C CNN
-	1    4800 1650
-	0    1    1    0
-$EndComp
-$Comp
 L Device:C C1
 U 1 1 5F3F49EA
 P 3850 2850
 F 0 "C1" V 3598 2850 50  0000 C CNN
-F 1 "C" V 3689 2850 50  0000 C CNN
+F 1 "0.35 pF" V 3689 2850 50  0000 C CNN
 F 2 "Resistor_SMD:R_0402_1005Metric" H 3888 2700 50  0001 C CNN
 F 3 "~" H 3850 2850 50  0001 C CNN
@@
 P 3850 3350
 F 0 "C2" V 3598 3350 50  0000 C CNN
-F 1 "C" V 3689 3350 50  0000 C CNN
+F 1 "0.1 pF" V 3689 3350 50  0000 C CNN
 F 2 "Resistor_SMD:R_0402_1005Metric" H 3888 3200 50  0001 C CNN
 F 3 "~" H 3850 3350 50  0001 C CNN
